Commit message: 

File: robot/ankbot/ankbot_description/urdf/ankbot.gazebo.xacro (robot description, xacro)
@@ -1,4 +1,4 @@
-<?xml version="1.0"?>
-<robot name="turtlebot3_waffle_sim" xmlns:xacro="http://ros.org/wiki/xacro">
+<?xml version="1.0" ?>
+<robot name="ankbot" xmlns:xacro="http://ros.org/wiki/xacro">
   <xacro:arg name="laser_visual"  default="false"/>
   <xacro:arg name="camera_visual" default="false"/>

File: robot/ankbot/ankbot_description/urdf/ankbot.urdf.xacro (robot description, xacro)
@@ -11,5 +11,5 @@
   <link name="base_link">
     <visual>
-      <origin xyz="0 0 0.06" rpy="0 0 -1.5707"/>
+      <origin xyz="0 0 0.062" rpy="0 0 1.5707"/>
       <geometry>
         <mesh filename="package://ankbot_description/meshes/robot_base.dae"/>

Commit message: 

File: robot/ankbot/ankbot_description/urdf/ankbot.gazebo.xacro (robot description, xacro)
@@ -5,5 +5,5 @@
   <xacro:arg name="imu_visual"    default="false"/>
   <gazebo reference="base_link">
-    <material>Gazebo/DarkGrey</material>
+    <material>Gazebo/LightBlack</material>
   </gazebo>
   <gazebo reference="wheel_left_link">
@@ -15,5 +15,5 @@
     <maxVel>0.1</maxVel>
     <fdir1>1 0 0</fdir1>
-    <material>Gazebo/FlatBlack</material>
+    <material>Gazebo/Black</material>
   </gazebo>
   <gazebo reference="wheel_right_link">
@@ -25,5 +25,5 @@
     <maxVel>0.1</maxVel>
     <fdir1>1 0 0</fdir1>
-    <material>Gazebo/FlatBlack</material>
+    <material>Gazebo/Black</material>
   </gazebo>
   <gazebo reference="caster_back_right_link">

File: robot/ankbot/ankbot_description/urdf/ankbot.urdf.xacro (robot description, xacro)
@@ -7,5 +7,5 @@
     <parent link="base_footprint"/>
     <child link="base_link"/>
-    <origin xyz="0 0 0.010" rpy="0 0 0"/>
+    <origin xyz="0 0 0.01" rpy="0 0 0"/>
   </joint>
   <link name="base_link">
@@ -129,5 +129,5 @@
     <parent link="base_link"/>
     <child link="imu_link"/>
-    <origin xyz="-0.032 0 0.068" rpy="0 0 0"/>
+    <origin xyz="-0.075 0 0.068" rpy="0 0 0"/>
   </joint>
   <link name="imu_link"/>
