Commit message: 

File: robot/ankbot/ankbot_description/urdf/ankbot.urdf.xacro (robot description, xacro)
@@ -129,5 +129,5 @@
     <parent link="base_link"/>
     <child link="imu_link"/>
-    <origin xyz="-0.075 0 0.068" rpy="0 0 0"/>
+    <origin xyz="0 -0.075 0.068" rpy="0 0 0"/>
   </joint>
   <link name="imu_link"/>

Commit message: 

File: robot/ankbot/ankbot_description/urdf/ankbot.urdf.xacro (robot description, xacro)
@@ -7,5 +7,5 @@
     <parent link="base_footprint"/>
     <child link="base_link"/>
-    <origin xyz="0 0 0.01" rpy="0 0 0"/>
+    <origin xyz="0 0 0.02" rpy="0 0 0"/>
   </joint>
   <link name="base_link">

Commit message: Config parameters

File: robot/ankbot/ankbot_description/urdf/ankbot.urdf.xacro (robot description, xacro)
@@ -7,5 +7,5 @@
     <parent link="base_footprint"/>
     <child link="base_link"/>
-    <origin xyz="0 0 0.02" rpy="0 0 0"/>
+    <origin xyz="0 0 0.01" rpy="0 0 0"/>
   </joint>
   <link name="base_link">
@@ -25,5 +25,5 @@
     <inertial>
       <origin xyz="0 0 0" rpy="0 0 0"/>
-      <mass value="8.2573504e-01"/>
+      <mass value="12.2573504e-01"/>
       <inertia ixx="2.2124416e-03" ixy="-1.2294101e-05" ixz="3.4938785e-05"
                iyy="2.1193702e-03" iyz="-5.0120904e-06"
@@ -89,5 +89,5 @@
     <parent link="base_link"/>
     <child link="caster_back_link"/>
-    <origin xyz="-0.081 0 -0.004" rpy="-1.57 0 0"/>
+    <origin xyz="-0.081 0 -0.0025" rpy="-1.57 0 0"/>
   </joint>
   <link name="caster_back_link">

Commit message: fix imu rpy

File: robot/ankbot/ankbot_description/urdf/ankbot.urdf.xacro (robot description, xacro)
@@ -129,5 +129,5 @@
     <parent link="base_link"/>
     <child link="imu_link"/>
-    <origin xyz="0 -0.075 0.068" rpy="0 0 0"/>
+    <origin xyz="0 -0.075 0.068" rpy="0 0 -1.5707"/>
   </joint>
   <link name="imu_link"/>

Commit message: update param

File: robot/ankbot/ankbot_description/urdf/ankbot.urdf.xacro (robot description, xacro)
@@ -129,5 +129,5 @@
     <parent link="base_link"/>
     <child link="imu_link"/>
-    <origin xyz="0 -0.075 0.068" rpy="0 0 -1.5707"/>
+    <origin xyz="0.07 -0.0025 0.12" rpy="0 0 0"/>
   </joint>
   <link name="imu_link"/>
